Commit message: 1. Removed the 5 m/s  limit of the car. That seems to have been there for a reason as the car just seems topple now.
2. Added params for easier testing

3. The car just starts flying even at slight turns for speeds greater than 5m/s. More mass and the damping and friction parameter seems to help. Need to test it more.  Modelling a suspension might be the longterm solution

File: urdf/macros.xacro (robot description, xacro)
@@ -4,8 +4,12 @@
   <xacro:arg name="robot_name" default="car_1" />
   <xacro:arg name="robot_skin" default="Blue" />
+  <!-- Wheel properties: Velocity in rad/s, damping in N∙m∙s/rad and friction in N∙m-->
+  <xacro:arg name="wheel_velocity" default="100" />
+  <xacro:arg name="wheel_damping" default="0" />
+  <xacro:arg name="wheel_friction" default="0" />
   <!-- inertial parameter macros -->
   <xacro:macro name="chassis_inertial_params">
     <origin xyz="0.1477 0 0" rpy="0 0 0" />
-    <mass value="4.0" />
+    <mass value="10.0" />
     <inertia ixx="0.010609" ixy="0"          ixz="0"
                             iyy="0.050409"   iyz="0"
@@ -161,5 +165,6 @@
     <child link="$(arg robot_name)_left_rear_wheel" />
     <axis xyz="0 0 -1" />
-    <limit effort="10" velocity="100" />
+    <limit effort="10" velocity="$(arg wheel_velocity)" />
+    <dynamics damping="$(arg wheel_damping)" friction="$(arg wheel_friction)"/>
   </joint>
   <xacro:wheel_transmission name="$(arg robot_name)_left_rear_wheel" />
@@ -182,5 +187,6 @@
     <child link="$(arg robot_name)_right_rear_wheel" />
     <axis xyz="0 0 -1" />
-    <limit effort="10" velocity="100" />
+    <limit effort="10" velocity="$(arg wheel_velocity)" />
+    <dynamics damping="$(arg wheel_damping)" friction="$(arg wheel_friction)"/>
   </joint>
   <xacro:wheel_transmission name="$(arg robot_name)_right_rear_wheel" />
@@ -239,5 +245,6 @@
     <child link="$(arg robot_name)_left_front_wheel" />
     <axis xyz="0 0 -1" />
-    <limit effort="10" velocity="100" />
+    <limit effort="10" velocity="$(arg wheel_velocity)" />
+    <dynamics damping="$(arg wheel_damping)" friction="$(arg wheel_friction)"/>
   </joint>
   <xacro:wheel_transmission name="$(arg robot_name)_left_front_wheel" />
@@ -260,5 +267,6 @@
     <child link="$(arg robot_name)_right_front_wheel" />
     <axis xyz="0 0 -1" />
-    <limit effort="10" velocity="100"/>
+    <limit effort="10" velocity="$(arg wheel_velocity)"/>
+    <dynamics damping="$(arg wheel_damping)" friction="$(arg wheel_friction)"/>
   </joint>
   <xacro:wheel_transmission name="$(arg robot_name)_right_front_wheel" />

Commit message: 1. Corrected the mass to 4. Adding friction to the ground plane prevents the car from taking off
2.  Converted the car to a 2 wheel drive

File: urdf/macros.xacro (robot description, xacro)
@@ -11,5 +11,5 @@
   <xacro:macro name="chassis_inertial_params">
     <origin xyz="0.1477 0 0" rpy="0 0 0" />
-    <mass value="10.0" />
+    <mass value="4.0" />
     <inertia ixx="0.010609" ixy="0"          ixz="0"
                             iyy="0.050409"   iyz="0"
@@ -248,5 +248,5 @@
     <dynamics damping="$(arg wheel_damping)" friction="$(arg wheel_friction)"/>
   </joint>
-  <xacro:wheel_transmission name="$(arg robot_name)_left_front_wheel" />
+  <!-- <xacro:wheel_transmission name="$(arg robot_name)_left_front_wheel" /> -->
   <!-- Add the left front wheel with its joints and tranmissions -->
   <link name="$(arg robot_name)_right_front_wheel">
@@ -270,5 +270,5 @@
     <dynamics damping="$(arg wheel_damping)" friction="$(arg wheel_friction)"/>
   </joint>
-  <xacro:wheel_transmission name="$(arg robot_name)_right_front_wheel" />
+  <!-- <xacro:wheel_transmission name="$(arg robot_name)_right_front_wheel" /> -->
   <!-- Add Hokuyo laser scanner -->
   <link name="$(arg robot_name)_laser">

Commit message: Tuned the car and the testing ground world to make the car perform as it does on vicon

File: urdf/macros.xacro (robot description, xacro)
@@ -8,4 +8,6 @@
   <xacro:arg name="wheel_damping" default="0" />
   <xacro:arg name="wheel_friction" default="0" />
+  <xacro:arg name="wheel_effort" default="5" />
+  <xacro:arg name="friction" default="1" />
   <!-- inertial parameter macros -->
   <xacro:macro name="chassis_inertial_params">
@@ -165,5 +167,5 @@
     <child link="$(arg robot_name)_left_rear_wheel" />
     <axis xyz="0 0 -1" />
-    <limit effort="10" velocity="$(arg wheel_velocity)" />
+    <limit effort="$(arg wheel_effort)" velocity="$(arg wheel_velocity)" />
     <dynamics damping="$(arg wheel_damping)" friction="$(arg wheel_friction)"/>
   </joint>
@@ -187,5 +189,5 @@
     <child link="$(arg robot_name)_right_rear_wheel" />
     <axis xyz="0 0 -1" />
-    <limit effort="10" velocity="$(arg wheel_velocity)" />
+    <limit effort="$(arg wheel_effort)" velocity="$(arg wheel_velocity)" />
     <dynamics damping="$(arg wheel_damping)" friction="$(arg wheel_friction)"/>
   </joint>
@@ -206,5 +208,5 @@
     <child link="$(arg robot_name)_left_steering_hinge" />
     <axis xyz="-1 0 0" />
-    <limit lower="-1.0" upper="1.0" effort="10" velocity="100" />
+    <limit lower="-1.0" upper="1.0" effort="0.88" velocity="100" />
   </joint>
   <xacro:steering_hinge_transmission name="$(arg robot_name)_left_steering_hinge" />
@@ -245,5 +247,5 @@
     <child link="$(arg robot_name)_left_front_wheel" />
     <axis xyz="0 0 -1" />
-    <limit effort="10" velocity="$(arg wheel_velocity)" />
+    <limit effort="$(arg wheel_effort)" velocity="$(arg wheel_velocity)" />
     <dynamics damping="$(arg wheel_damping)" friction="$(arg wheel_friction)"/>
   </joint>
@@ -267,5 +269,5 @@
     <child link="$(arg robot_name)_right_front_wheel" />
     <axis xyz="0 0 -1" />
-    <limit effort="10" velocity="$(arg wheel_velocity)"/>
+    <limit effort="$(arg wheel_effort)" velocity="$(arg wheel_velocity)"/>
     <dynamics damping="$(arg wheel_damping)" friction="$(arg wheel_friction)"/>
   </joint>
@@ -360,6 +362,6 @@
   </gazebo>
   <gazebo reference="$(arg robot_name)_left_rear_wheel">
-    <mu1 value="1.0"/>
-    <mu2 value="1.0"/>
+    <mu1 value="$(arg friction)"/>
+    <mu2 value="$(arg friction)"/>
     <kp  value="10000000.0" />
     <kd  value="1.0" />
@@ -368,6 +370,6 @@
   </gazebo>
   <gazebo reference="$(arg robot_name)_right_rear_wheel">
-    <mu1 value="1.0"/>
-    <mu2 value="1.0"/>
+    <mu1 value="$(arg friction)"/>
+    <mu2 value="$(arg friction)"/>
     <kp  value="10000000.0" />
     <kd  value="1.0" />
@@ -376,6 +378,6 @@
   </gazebo>
   <gazebo reference="$(arg robot_name)_left_front_wheel">
-    <mu1 value="1.0"/>
-    <mu2 value="1.0"/>
+    <mu1 value="$(arg friction)"/>
+    <mu2 value="$(arg friction)"/>
     <kp  value="10000000.0" />
     <kd  value="1.0" />
@@ -384,6 +386,6 @@
   </gazebo>
   <gazebo reference="$(arg robot_name)_right_front_wheel">
-    <mu1 value="1.0"/>
-    <mu2 value="1.0"/>
+    <mu1 value="$(arg friction)"/>
+    <mu2 value="$(arg friction)"/>
     <kp  value="10000000.0" />
     <kd  value="1.0" />

Commit message: Fined tuned the friction and effort values. Added a param for the hinge effort

File: urdf/macros.xacro (robot description, xacro)
@@ -9,4 +9,5 @@
   <xacro:arg name="wheel_friction" default="0" />
   <xacro:arg name="wheel_effort" default="5" />
+  <xacro:arg name="hinge_effort" default="0.88" />
   <xacro:arg name="friction" default="1" />
   <!-- inertial parameter macros -->
@@ -208,5 +209,5 @@
     <child link="$(arg robot_name)_left_steering_hinge" />
     <axis xyz="-1 0 0" />
-    <limit lower="-1.0" upper="1.0" effort="0.88" velocity="100" />
+    <limit lower="-1.0" upper="1.0" effort="$(arg hinge_effort)" velocity="100" />
   </joint>
   <xacro:steering_hinge_transmission name="$(arg robot_name)_left_steering_hinge" />
@@ -226,5 +227,5 @@
     <child link="$(arg robot_name)_right_steering_hinge" />
     <axis xyz="-1 0 0" />
-    <limit lower="-1.0" upper="1.0" effort="10" velocity="100" />
+    <limit lower="-1.0" upper="1.0" effort="$(arg hinge_effort)" velocity="100" />
   </joint>
   <xacro:steering_hinge_transmission name="$(arg robot_name)_right_steering_hinge" />

Commit message: remove unused and unneeded

File: urdf/macros.xacro (robot description, xacro)
@@ -51,5 +51,5 @@
     <origin xyz="0.46 -0.135 -0.180" rpy="1.57 0 3.14" />
     <geometry>
-      <mesh filename="package://f1tenth-sim/urdf/meshes/chassis.stl" scale="0.000990 0.0009375 0.0009375"/>
+      <mesh filename="package://audubon-gazebo/urdf/meshes/chassis.stl" scale="0.000990 0.0009375 0.0009375"/>
     </geometry>
   </xacro:macro>
@@ -57,5 +57,5 @@
     <origin xyz="0 0 0" rpy="0 0 0" />
     <geometry>
-      <mesh filename="package://f1tenth-sim/urdf/meshes/left_wheel.stl" />
+      <mesh filename="package://audubon-gazebo/urdf/meshes/left_wheel.stl" />
     </geometry>
   </xacro:macro>
@@ -63,5 +63,5 @@
     <origin xyz="0 0 0" rpy="0 0 0" />
     <geometry>
-      <mesh filename="package://f1tenth-sim/urdf/meshes/right_wheel.stl" />
+      <mesh filename="package://audubon-gazebo/urdf/meshes/right_wheel.stl" />
     </geometry>
   </xacro:macro>
@@ -69,5 +69,5 @@
     <origin xyz="0 0 0" rpy="0 0 0" />
     <geometry>
-      <mesh filename="package://f1tenth-sim/urdf/meshes/left_wheel.stl" />
+      <mesh filename="package://audubon-gazebo/urdf/meshes/left_wheel.stl" />
     </geometry>
   </xacro:macro>
@@ -75,5 +75,5 @@
     <origin xyz="0 0 0" rpy="0 0 0" />
     <geometry>
-      <mesh filename="package://f1tenth-sim/urdf/meshes/right_wheel.stl" />
+      <mesh filename="package://audubon-gazebo/urdf/meshes/right_wheel.stl" />
     </geometry>
   </xacro:macro>
@@ -81,5 +81,5 @@
     <origin xyz="0 0 0" rpy="0 0 0" />
     <geometry>
-      <mesh filename="package://f1tenth-sim/urdf/meshes/hinge.stl" />
+      <mesh filename="package://audubon-gazebo/urdf/meshes/hinge.stl" />
     </geometry>
   </xacro:macro>
@@ -87,5 +87,5 @@
     <origin xyz="0 0 0" rpy="0 0 0" />
     <geometry>
-      <mesh filename="package://f1tenth-sim/urdf/meshes/hinge.stl" />
+      <mesh filename="package://audubon-gazebo/urdf/meshes/hinge.stl" />
     </geometry>
   </xacro:macro>
@@ -288,5 +288,5 @@
       <origin xyz="0 0 0" rpy="0 0 0"/>
       <geometry>
-        <mesh filename="package://f1tenth-sim/urdf/meshes/hokuyo.stl"/>
+        <mesh filename="package://audubon-gazebo/urdf/meshes/hokuyo.stl"/>
         <material name="grey" />
       </geometry>

Commit message: Moved the hokyuo to the front and added an imu to it. It does not see the chassis behind it because the chassis has no colission geometry.

File: urdf/macros.xacro (robot description, xacro)
@@ -294,5 +294,7 @@
   </link>
   <joint name="$(arg robot_name)_hokuyo_joint" type="fixed">
-    <origin xyz="0.125 0.0 0.155" rpy="0 0 0"/>
+    <origin xyz="0.390 0 0.070" rpy="0 0 0"/>
+    <!-- The commented config is to place the hokuyo on top -->
+    <!-- <origin xyz="0.125 0.0 0.155" rpy="0 0 0"/> -->
     <parent link="$(arg robot_name)_chassis" />
     <child link="$(arg robot_name)_laser" />
@@ -300,5 +302,5 @@
   </joint>
   <!-- camera class (spawn parameters) -->
-  <link name="$(arg robot_name)_link">
+  <!-- <link name="$(arg robot_name)_link">
     <inertial>
       <mass value="1e-5" />
@@ -319,14 +321,13 @@
       <material name="red"/>
     </visual>
-  </link>
-  <joint name="$(arg robot_name)_joint" type="fixed">
+  </link> -->
+  <!-- <joint name="$(arg robot_name)_joint" type="fixed">
     <origin xyz="0.390 0 0.025" rpy="0 0 0"/>
     <parent link="$(arg robot_name)_chassis"/>
     <child link="$(arg robot_name)_link"/>
     <axis xyz="0 0 1" />
-    <!-- <limit lower="0.0" upper="0.0" effort="0.0" velocity="0.0" /> -->
-  </joint>
+  </joint> -->
   <!-- camera lenses -->
-  <link name="$(arg robot_name)_camera_link">
+  <!-- <link name="$(arg robot_name)_camera_link">
     <inertial>
       <mass value="1e-5" />
@@ -353,5 +354,5 @@
     <child link="$(arg robot_name)_right_link"/>
     <axis xyz="0 0 1" />
-  </joint>
+  </joint> -->
   <!-- Gazebo references -->
   <gazebo reference="$(arg robot_name)_chassis">
@@ -446,4 +447,18 @@
         </plugin>
       </sensor>
+    </gazebo>
+    <gazebo>
+      <plugin name="imu_controller" filename="libhector_gazebo_ros_imu.so">
+        <!-- <robotNamespace>$(arg robot_namespace)</robotNamespace> -->
+        <updateRate>50.0</updateRate>
+        <bodyName>$(arg robot_name)_laser</bodyName>
+        <topicName>$(arg robot_name)_laser_imu</topicName>
+        <accelDrift>0.005 0.005 0.005</accelDrift>
+        <accelGaussianNoise>0.005 0.005 0.005</accelGaussianNoise>
+        <rateDrift>0.005 0.005 0.005 </rateDrift>
+        <rateGaussianNoise>0.005 0.005 0.005 </rateGaussianNoise>
+        <headingDrift>0.005</headingDrift>
+        <headingGaussianNoise>0.005</headingGaussianNoise>
+      </plugin>
     </gazebo>
   </xacro:unless>

Commit message: Added a stereo camera with IMU. Removed old unused plugins

File: urdf/macros.xacro (robot description, xacro)
@@ -302,5 +302,5 @@
   </joint>
   <!-- camera class (spawn parameters) -->
-  <!-- <link name="$(arg robot_name)_link">
+  <link name="$(arg robot_name)_camera_link">
     <inertial>
       <mass value="1e-5" />
@@ -321,38 +321,11 @@
       <material name="red"/>
     </visual>
-  </link> -->
-  <!-- <joint name="$(arg robot_name)_joint" type="fixed">
-    <origin xyz="0.390 0 0.025" rpy="0 0 0"/>
+  </link>
+  <joint name="$(arg robot_name)_camera_joint" type="fixed">
+    <origin xyz="0.415 0 0.1" rpy="0 0 0"/>
     <parent link="$(arg robot_name)_chassis"/>
-    <child link="$(arg robot_name)_link"/>
-    <axis xyz="0 0 1" />
-  </joint> -->
-  <!-- camera lenses -->
-  <!-- <link name="$(arg robot_name)_camera_link">
-    <inertial>
-      <mass value="1e-5" />
-      <origin xyz="-2.5 0 1.75" rpy="0 .57 0"/>
-      <inertia ixx="1e-6" ixy="0" ixz="0" iyy="1e-6" iyz="0" izz="1e-6" />
-    </inertial>
-  </link>
-  <link name="$(arg robot_name)_right_link">
-    <inertial>
-      <mass value="1e-5" />
-      <origin xyz="-2.5 0 1.75" rpy="0 .57 0"/>
-      <inertia ixx="1e-6" ixy="0" ixz="0" iyy="1e-6" iyz="0" izz="1e-6" />
-    </inertial>
-  </link>
-  <joint name="$(arg robot_name)_left_joint" type="fixed">
-    <origin xyz="-2.5 0 1.75" rpy="0 .57 0"/>
-    <parent link="$(arg robot_name)_link"/>
     <child link="$(arg robot_name)_camera_link"/>
     <axis xyz="0 0 1" />
   </joint>
-  <joint name="$(arg robot_name)_right_joint" type="fixed">
-    <origin xyz="0 -0.06 0.025" rpy="0 0 0"/>
-    <parent link="$(arg robot_name)_link"/>
-    <child link="$(arg robot_name)_right_link"/>
-    <axis xyz="0 0 1" />
-  </joint> -->
   <!-- Gazebo references -->
   <gazebo reference="$(arg robot_name)_chassis">
@@ -450,8 +423,7 @@
     <gazebo>
       <plugin name="imu_controller" filename="libhector_gazebo_ros_imu.so">
-        <!-- <robotNamespace>$(arg robot_namespace)</robotNamespace> -->
-        <updateRate>50.0</updateRate>
+        <updateRate>40.0</updateRate>
         <bodyName>$(arg robot_name)_laser</bodyName>
-        <topicName>$(arg robot_name)_laser_imu</topicName>
+        <topicName>$(arg robot_name)/laser/imu</topicName>
         <accelDrift>0.005 0.005 0.005</accelDrift>
         <accelGaussianNoise>0.005 0.005 0.005</accelGaussianNoise>
@@ -464,16 +436,14 @@
   </xacro:unless>
   <!-- camera object -->
-  <!-- <xacro:unless value="$(optenv DISABLE_GAZEBO_CAMERA false)">
+  <xacro:unless value="$(optenv DISABLE_GAZEBO_CAMERA false)">
     <gazebo reference="$(arg robot_name)_camera_link">
-      <sensor type="camera" name="$(arg robot_name)_left_sensor">
-        <update_rate>30.0</update_rate> -->
-        <!-- math.atan(320 / 687.8065795898438) * 2 COMMENT -->
-        <!-- <camera name="front_camera"> -->
-          <!-- horizontal_fov>0.8709216071359963</horizontal_fov COMMENT-->
-          <!-- <horizontal_fov>1.74</horizontal_fov>
+      <sensor type="multicamera" name="stereo_camera">
+        <update_rate>30.0</update_rate>
+        <camera name="left">
+          <horizontal_fov>1.3962634</horizontal_fov>
           <image>
-            <width>1920</width>
-            <height>1080</height>
-            <format>B8G8R8</format>
+            <width>800</width>
+            <height>800</height>
+            <format>R8G8B8</format>
           </image>
           <clip>
@@ -487,13 +457,30 @@
           </noise>
         </camera>
-        <plugin name="camera_controller" filename="libgazebo_ros_camera.so">
+        <camera name="right">
+          <pose>0 -0.07 0 0 0 0</pose>
+          <horizontal_fov>1.3962634</horizontal_fov>
+          <image>
+            <width>800</width>
+            <height>800</height>
+            <format>R8G8B8</format>
+          </image>
+          <clip>
+            <near>0.02</near>
+            <far>300</far>
+          </clip>
+          <noise>
+            <type>gaussian</type>
+            <mean>0.0</mean>
+            <stddev>0.007</stddev>
+          </noise>
+        </camera>
+        <plugin name="stereo_camera_controller" filename="libgazebo_ros_multicamera.so">
           <alwaysOn>true</alwaysOn>
-          <updateRate>30.0</updateRate>
-          <cameraName>/$(arg robot_name)/camera</cameraName>
-          <imageTopicName>image</imageTopicName>
-          <cameraInfoTopicName>rgb/camera_info</cameraInfoTopicName>
-          <frameName>$(arg robot_name)_camera_link</frameName> -->
-          <!-- set this to 0.12 for the second camera  COMMENT -->
-          <!-- <hackBaseline>0</hackBaseline>
+          <updateRate>0.0</updateRate>
+          <cameraName>$(arg robot_name)/camera</cameraName>
+          <imageTopicName>image_raw</imageTopicName>
+          <cameraInfoTopicName>camera_info</cameraInfoTopicName>
+          <frameName>left_camera_optical_frame</frameName>
+          <hackBaseline>0.07</hackBaseline>
           <distortionK1>0.0</distortionK1>
           <distortionK2>0.0</distortionK2>
@@ -504,5 +491,18 @@
       </sensor>
     </gazebo>
-  </xacro:unless> -->
+    <gazebo>
+      <plugin name="imu_controller" filename="libhector_gazebo_ros_imu.so">
+        <updateRate>30.0</updateRate>
+        <bodyName>$(arg robot_name)_camera_link</bodyName>
+        <topicName>$(arg robot_name)/camera/imu</topicName>
+        <accelDrift>0.005 0.005 0.005</accelDrift>
+        <accelGaussianNoise>0.005 0.005 0.005</accelGaussianNoise>
+        <rateDrift>0.005 0.005 0.005 </rateDrift>
+        <rateGaussianNoise>0.005 0.005 0.005 </rateGaussianNoise>
+        <headingDrift>0.005</headingDrift>
+        <headingGaussianNoise>0.005</headingGaussianNoise>
+      </plugin>
+    </gazebo>
+  </xacro:unless>
   <material name="black">
     <color rgba="0.0 0.0 0.0 1.0"/>
